File: Hardware/0. Project/AC-DC.brd (EAGLE design)
At the start: 100 x 75 mm, 107 parts, among them IC1 LM393D, IC2 LM393D, IC3 LM358D, K1 12VDC COIL, K2 12VDC COIL, K3 12VDC COIL, K4 12VDC COIL, Q1 BC848, Q2 BC848, Q3 BC858, Q4 BC848, Q5 BC858, Q6 BC858, U1 LM338K, U2 HLK-PM01, U3 LM338K

Commit message: Schematic and PCB layout 2.1 updated
Parts:
- removed IC1, IC2: LM393D, linear:SO08
- removed IC3: LM358D, linear:SO08
- removed OK1, OK2, OK3, OK4: 4N33, optocoupler:DIL6-SMD
- added U10: (no value), REG1117:MOLEX3P
- added U4, U8, U9: 4N33, optocoupler:DIL6-SMD
- added U5: (no value), HLK-PM01:HLK-PM01
- added U6: LM393D, linear:SO08
- added U7: LM358D, linear:SO08
- AMP1, AMP2: value AMMETER -> (none)
- B1, B2: value KBPC608 -> (none)
- C1: value 15.000uF x 50V -> (none)
- C10, C14, C3: value 10uF x 50V -> (none); device rcl:153CLV-0605 -> rcl:C0805
- C11, C2: value 100nF x 50V -> (none)
- C12, C15, C5, C8: value 100nF x 50V -> (none); device rcl:C0805 -> rcl:153CLV-0605
- C13, C4, C6: value 10uF x 50V -> (none)
- C7: value 15.000uF x 50V -> (none); device rcl:EB35D -> rcl:C0805
- C9: value 10uF x 50V -> (none); device rcl:153CLV-0605 -> rcl:EB35D
- D1, D5: value 12V / 0.5W -> (none)
- D10, D11, D4, D8, D9: value 1N4148 -> (none)
- D2, D3, D6, D7: value 1N4007 -> (none)
- K1, K2, K3, K4: value 12VDC COIL -> (none)
- L1: value MOTOR -> (none)
- LED1: value Bicolor LED Common-Anode -> (none)
- Q1, Q2, Q4: value BC848 -> (none)
- Q3, Q5, Q6: value BC858 -> (none)
- R1, R16, R17, R2: value 500k -> (none); device rcl:RTRIM64W -> rcl:RTRIM3202
- R10, R27: value 5K -> (none); device trimpot-molex2p:MOLEX3P -> rcl:R0805
- R11, R28, R34, R36: value 1k (5%) -> (none)
- R12, R29, R44: value 100k (5%) -> (none)
- R13, R30: value 1k (5%) -> (none); device rcl:R0805 -> rcl:RTRIM3202
- R14, R31: value 100k (5%) -> (none); device rcl:R0805 -> trimpot-molex2p:MOLEX3P
- R15, R23, R24, R32, R33, R35, R39, R42, R45, R7, R8: value 10k (5%) -> (none)
- R18, R37, R38, R4, R40, R41: value 100k (1%) -> (none)
- R19, R21: value 10k -> (none); device rcl:RTRIM64W -> rcl:RTRIM3202
- R20, R5: value 33k (1%) -> (none)
- R22, R6: value 220R -> (none)
- R25: value 33k (5%) -> (none)
- R26, R9: value 500R -> (none); device pot:CA6V -> rcl:R0805
- R43: value 220k (5%) -> (none)
- RT1, RT2: value 5R -> (none)
- RT3: value 10k -> (none)
- TR1, TR2: value 24VRMS -> (none)
- U1: value LM338K -> LM393D; device REG1117:MOLEX3P -> linear:SO08
- U2: value HLK-PM01 -> (none); device HLK-PM01:HLK-PM01 -> REG1117:MOLEX3P
- U3: value LM338K -> 4N33; device REG1117:MOLEX3P -> optocoupler:DIL6-SMD
- VOLT1, VOLT2: value VOLTMETER -> (none)
- moved D5 200.2 mm to (78.7, 69.6), turned to 90 degrees
- moved C12 198.0 mm to (73.7, 69.3), turned to 270 degrees
- moved R20 195.3 mm to (49.9, 54.7), turned to 90 degrees
- moved R22 190.2 mm to (68.1, 69.5), turned to 270 degrees
- moved C14 188.0 mm to (85.3, 45.7), turned to 90 degrees
- moved R18 187.9 mm to (49.9, 58.9), turned to 90 degrees
- moved C15 172.0 mm to (62.4, 69.4), turned to 270 degrees
- moved R23 168.2 mm to (41.7, 63.7), turned to 270 degrees
- moved R8 165.6 mm to (72.2, 20.1), turned to 90 degrees
- moved C11 162.9 mm to (41.7, 59.9), turned to 90 degrees
- moved R24 160.0 mm to (43.4, 55.4), turned to 270 degrees
- moved R14 130.3 mm to (44.5, 3.42), flipped to the top, turned to 180 degrees
- moved R13 125.2 mm to (34.8, 9.33), turned to 0 degrees
- moved R7 121.7 mm to (49.4, 18.9), turned to 90 degrees
- moved R5 120.2 mm to (43.2, 19.0), turned to 270 degrees
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Connections:
- removed net 0V: C11.2, C12.2
- net !SHORT_CIRCUIT_DETECTED!: now also R12.2, R29.2, U4.4, U9.4; no longer OK2.4, OK4.4, R14.2, R31.2
- net !VOUT1_POWER_ON!: now also U7.6; no longer IC3.6
- net !VOUT1_POWER_ON!1: now also R11.1, U4.5; no longer OK2.5, R13.1
- net !VOUT1_POWER_ON!2: now also R9.1, U3.5; no longer OK1.5, R11.1
- net !VOUT1_POWER_ON!3: now also R28.1, U9.5; no longer OK4.5, R30.1
- net !VOUT1_POWER_ON!4: now also R26.1, U8.5; no longer OK3.5, R28.1
- net !VOUT_POWER_OFF!: now also U7.7; no longer IC3.7
- net +12V: now also C14.1, C7.1, C8.+, R26.2, R9.2, U5.P$4, U7.8; no longer C15.1, C5.1, C6.+, IC3.8, R13.2, R30.2, U2.P$4
- net 0V_B: now also U5.P$2, X1.2; no longer U2.P$2, X3.2
- net 127V_B: now also U5.P$1, X1.1; no longer U2.P$1, X3.1
- net 12V_AUX1: now also C3.1, C4.+, U1.8; no longer C11.1, C13.+, IC1.8
- net 12V_AUX2: now also C11.1, C12.+, U6.8; no longer C12.1, C14.+, IC2.8
- net C_FULL_1: now also U2.1; no longer U1.1
- net C_FULL_2: now also C10.1, C9.+, U10.1; no longer C7.+, C8.1, U3.1
- net GND1: now also C3.2, C5.-, C6.-, R14.P$1, R14.P$3, U1.4, U3.2, U4.2, X2.2; no longer C13.-, C3.-, IC1.4, OK1.2, OK2.2, R10.P$1, R10.P$3, X1.2
- net GND2: now also C10.2, C11.2, C12.-, C13.-, C15.-, R31.P$1, R31.P$3, U6.4, U8.2, U9.2, X3.2; no longer C10.-, C14.-, C7.-, C8.2, IC2.4, OK3.2, OK4.2, R27.P$1, R27.P$3, X2.2
- net HIGH_TEMPERATURE: now also U7.1; no longer IC3.1
- net N$12: now also D9.C; no longer D10.C
- net N$15: now also C6.+, R13.3, U2.3; no longer C4.+, R9.E, U1.3
- net N$16: now also C5.+, R13.1, R13.2, R14.P$2, U2.2; no longer C3.+, R10.P$2, R9.A, R9.S, U1.2
- net N$17: now also X2.1; no longer X1.1
- net N$18: now also U1.5; no longer IC1.5
- net N$19: now also R7.1, U1.1; no longer IC1.1, R8.1
- net N$20: now also R7.2, U4.1; no longer OK2.1, R8.2
- net N$21: now also U7.5; no longer IC3.5
- net N$25: now also U1.2; no longer IC1.2
- net N$26: now also C15.+, R30.3, U10.3; no longer C10.+, R26.E, U3.3
- net N$27: now also C13.+, R30.1, R30.2, R31.P$2, U10.2; no longer C9.+, R26.A, R26.S, R27.P$2, U3.2
- net N$28: now also X3.1; no longer X2.1
- net N$35: now also U7.2; no longer IC3.2
- net N$36: now also U7.3; no longer IC3.3
- net N$37: now also R8.1, U1.7; no longer IC1.7, R7.1
- net N$38: now also D10.C; no longer D9.C
- net N$39: now also R8.2, U3.1; no longer OK1.1, R7.2
- net N$41: now also U6.5; no longer IC2.5
- net N$42: now also R23.1, U6.1; no longer IC2.1, R24.1
- net N$43: now also U6.6; no longer IC2.6
- net N$44: now also R23.2, U9.1; no longer OK4.1, R24.2
- net N$45: now also R24.1, U6.7; no longer IC2.7, R23.1
- net N$46: now also R24.2, U8.1; no longer OK3.1, R23.2
- net N$47: now also R27.2, U8.4; no longer OK3.4, R29.2
- net N$48: now also R10.2, U3.4; no longer OK1.4, R12.2
- net N$5: now also U6.2; no longer IC2.2
- net N$6: now also U1.6; no longer IC1.6
- net PE: now also C14.2, C7.2, C8.-, R10.1, R27.1, U5.P$3, U7.4; no longer C15.2, C5.2, C6.-, IC3.4, R14.1, R31.1, U2.P$3
- net VOUT_1: now also U1.3; no longer IC1.3, IC2.3
- net VOUT_2: now also U6.3
Routing:
- net +12V: track 0.00 -> 200.1 mm, vias 0 -> 5
- net 12V_AUX2: track 0.00 -> 99.4 mm, vias 0 -> 2
- net 12V_AUX1: track 0.00 -> 97.2 mm
- net PE: track 0.00 -> 78.4 mm, vias 0 -> 64
- net N$33: track 0.00 -> 69.7 mm
- net N$2: track 0.00 -> 61.9 mm, vias 0 -> 2
- net N$12: track 0.00 -> 60.2 mm, vias 0 -> 3
- net !SHORT_CIRCUIT_DETECTED!: track 0.00 -> 53.9 mm, vias 0 -> 2
- net VOUT_2: track 20.9 -> 74.6 mm
- net C_FULL_2: track 25.9 -> 78.6 mm, vias 0 -> 2
- net VOUT_1: track 20.9 -> 68.4 mm, vias 0 -> 2
- net N$27: track 0.00 -> 39.3 mm
- net N$16: track 0.00 -> 37.0 mm
- net !VOUT_POWER_OFF!: track 0.00 -> 35.8 mm, vias 0 -> 3
- net C_FULL_1: track 38.6 -> 74.0 mm, vias 0 -> 4
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- added copper zone on layer 1, net GND1
- added copper zone on layer 16, net GND1
- added copper zone on layer 1, net GND2
- added copper zone on layer 16, net GND2
- added copper zone on layer 1, net PE
- added copper zone on layer 16, net PE
Other:
- board text added: "AC 127V 220V"
