File: Hardware/0. Project/AC-DC.brd (EAGLE design)
At the start: 100 x 75 mm, 107 parts, among them U1 LM393D, U3 4N33, U4 4N33, U6 LM393D, U7 LM358D, U8 4N33, U9 4N33

Commit message: File updated to 2.2 PCB rev.
Parts:
- B1, B2: value (none) -> KBPC608
- C1, C9: value (none) -> 15.000uF x 50V
- C10, C11, C14, C2, C3, C7: value (none) -> 100nF x 50V
- C12, C13, C15, C4, C5, C6, C8: value (none) -> 10uF x 50V
- D1, D5: value (none) -> 12V / 0.5W
- D10, D11, D4, D8, D9: value (none) -> 1N4148
- D2, D3, D6, D7: value (none) -> 1N4007
- L1: value (none) -> FAN Cooler
- Q1, Q2, Q4: value (none) -> BC817
- Q3, Q5, Q6: value (none) -> BC807
- R1, R16, R17, R2: value (none) -> 100k
- R10, R12, R18, R27, R29, R4, R44: value (none) -> 100k (5%)
- R11, R26, R28, R34, R36, R9: value (none) -> 1k (5%)
- R13, R30: value (none) -> 1k
- R14, R31: value (none) -> 5k
- R15, R23, R24, R32, R33, R35, R39, R42, R45, R7, R8: value (none) -> 10k (5%)
- R19, R21, RT3: value (none) -> 10k
- R20, R25, R5: value (none) -> 33k (5%)
- R22, R6: value (none) -> 220R (5%)
- R37, R38, R40, R41: value (none) -> 100k (1%)
- R43: value (none) -> 220k (5%)
- RT1, RT2: value (none) -> 5R
- TR1, TR2: value (none) -> 24VRMS / 5A
- U10, U2: value (none) -> LM338K
- U5: value (none) -> HLK-PM01
