File: Hardware/0. Project/AC-DC.sch (EAGLE design)
At the start: 92 parts, among them IC1 7812TV, IC2 7824TV, IC3 LM324N, IC4 LM358N, K1 APF30212C, K2 12VDC, K3 12VDC, K4 12VDC, K5 APF30212C, K7 12VDC, Q1 BC548B, Q2 BC558B, Q3 BC558B, Q4 BC558B, Q5 BC558B, SW1 CT10-XXXX-A2, T1 BC337, U1 LM338K, U2 LM338K

Commit message: Schematic updated to 1.1 version
Parts:
- removed C14: 10uF x 50V, rcl:CPOL-EUE3.5-8
- removed D10, D2, D3: 1N4007, diode:1N5060GP
- removed K7: 12VDC, relay:APF30212C
- removed L2: Cooler 24V @ 6W, Inductor:INDUCTOR
- added C1: 100nF x 50V, rcl:C-EU025-025X050
- added D9: 1N4007, diode:1N5060GP
- added K6: 12VDC, relay:APF30212C
- added L1: Cooler 24V @ 6W, Inductor:INDUCTOR
- added R35, R36: 1k (5%), rcl:R-EU_0207/7
- added R37, R38: 10k (5%), rcl:R-EU_0207/7
- C10, C6: value 10uF x 50V -> 15.000uF x 50V; device rcl:CPOL-EUE3.5-8 -> rcl:CPOL-EUE10-35
- C11, C7: value 10uF x 50V -> 100nF x 50V; device rcl:CPOL-EUE3.5-8 -> rcl:C-EU025-025X050
- C12, C13, C5, C9: value 100nF x 50V -> 10uF x 50V; device rcl:C-EU025-025X050 -> rcl:CPOL-EUE3.5-8
- C4: value 15.000uF x 50V -> 100nF x 50V; device rcl:CPOL-EUE10-35 -> rcl:C-EU025-025X050
- C8: value 15.000uF x 50V -> 10uF x 50V; device rcl:CPOL-EUE10-35 -> rcl:CPOL-EUE3.5-8
- IC1: value 7812TV -> 7824TV; device linear:7812TV -> linear:7824TV
- IC2: value 7824TV -> 7812TV; device linear:7824TV -> linear:7812TV
- K1: value APF30212C -> 12VDC
- K3: value 12VDC -> APF30212C
- R1: value VARISTOR-2,5 -> 500k; device varistor:VARISTOR-2,5 -> rcl:R-TRIMM64W
- R10: value 220k (5%) -> 10k; device rcl:R-EU_0207/7 -> ptc-ntc:NTC640
- R11: value 1k (5%) -> 10k; device rcl:R-EU_0207/7 -> rcl:R-TRIMM64W
- R12: value 10k (5%) -> 500R; device rcl:R-EU_0207/7 -> rcl:R-TRIMMT93YB
- R13: value 100R (5%) -> 5K; device rcl:R-EU_0207/7 -> pot:3RP/1610N
- R14: value 5R -> 33k (5%); device ptc-ntc:NTC640 -> rcl:R-EU_0207/7
- R15: value 10k (5%) -> 10k; device rcl:R-EU_0207/7 -> rcl:R-TRIMM64W
- R16, R26, R29, R34: value 100k (5%) -> 10k (5%)
- R17, R18: value 10k (5%) -> 100k (1%)
- R19: value 500k -> 10k; device rcl:R-TRIMM64W -> ptc-ntc:NTC640
- R2: value 500k -> VARISTOR-2,5; device rcl:R-TRIMM64W -> varistor:VARISTOR-2,5
- R20, R9: value 100k (1%) -> 10k; device rcl:R-EU_0207/7 -> rcl:R-TRIMM64W
- R21: value 33k (1%) -> 100k (1%)
- R22: value 5K -> 100k (1%); device pot:3RP/1610N -> rcl:R-EU_0207/7
- R23: value 500R -> 33k (5%); device rcl:R-TRIMMT93YB -> rcl:R-EU_0207/7
- R24: value 5R -> 220k (5%); device ptc-ntc:NTC640 -> rcl:R-EU_0207/7
- R25: value 100k (5%) -> 5R; device rcl:R-EU_0207/7 -> ptc-ntc:NTC640
- R27: value 10k -> 1k (5%); device ptc-ntc:NTC640 -> rcl:R-EU_0207/7
- R28: value 10k -> 10k (5%); device ptc-ntc:NTC640 -> rcl:R-EU_0207/7
- R3: value 500R -> 100k (1%); device rcl:R-TRIMMT93YB -> rcl:R-EU_0207/7
- R30: value 10k -> 500R; device rcl:R-TRIMM64W -> rcl:R-TRIMMT93YB
- R31: value 10k -> 5K; device rcl:R-TRIMM64W -> pot:3RP/1610N
- R32: value 10k -> 1k (5%); device rcl:R-TRIMM64W -> rcl:R-EU_0207/7
- R33: value 10k -> 100k (5%); device rcl:R-TRIMM64W -> rcl:R-EU_0207/7
- R4: value 5K -> 33k (1%); device pot:3RP/1610N -> rcl:R-EU_0207/7
- R6: value 100k (1%) -> 10k (5%)
- R7: value 100k (1%) -> 500k; device rcl:R-EU_0207/7 -> rcl:R-TRIMM64W
- R8: value 100k (1%) -> 5R; device rcl:R-EU_0207/7 -> ptc-ntc:NTC640
Connections:
- removed net N$7 (its old number): Q3.B, R17.2
- new net N$32: Q3.B, R28.2
- net !SHORT_CIRCUIT_DETECTED!: now also R35.2, R36.2; no longer D3.C, D4.C
- net !VOUT1_POWER_OFF!: now also R24.2, R27.2, R33.1, R34.1; no longer R10.2, R11.2, R17.1, R5.1
- net !VOUT1_POWER_ON!: now also R17.1, R18.2, R26.2; no longer R12.2, R6.1, R7.2
- net +24V: now also C2.1, C3.+, D1.C, IC1.VO, IC2.VI, K11.1, K21.1, Q3.E, R1.E, R10.2, R15.E, R19.2, R3.2, R37.2, R38.2, R9.E; no longer C12.1, C14.+, D6.C, IC1.VI, IC2.VO, K41.1, K71.1, Q5.E, R19.E, R20.2, R27.2, R28.2, R31.E, R33.E
- net 0V: now also C1.2, C11.2, C12.-, C13.-, C4.2, C5.-, C7.2, C9.-, D8.A, D9.A, K41.2, K61.2, L1.2, R1.A, R11.A, R13.A, R13.S, R15.A, R20.A, R22.1, R31.S, R33.2, R4.1, R5.1, R7.A, R9.A; no longer C11.-, C12.2, C13.2, C14.-, C4.-, C5.2, C7.-, C9.2, D10.A, D7.A, K21.2, K31.2, L2.2, R19.A, R2.A, R21.1, R22.A, R22.S, R30.A, R32.A, R33.A, R4.A, R4.S, R7.1, R9.1
- net 0V_A: now also R2.2; no longer R1.2
- net 127V_A: now also R2.1; no longer R1.1
- net 12V: now also C4.1, C5.+, IC2.VO, Q5.E, R17.2, R21.2, R7.E; no longer C2.1, C3.+, IC1.VO, Q3.E, R16.2, R2.E, R6.2, R8.2
- net 30V: now also C1.1, C10.+, C11.1, C6.+, C7.1, D4.C, D6.C, IC1.VI, K12.S, K22.S, R25.1, R8.1; no longer C13.1, C4.+, C5.1, C8.+, C9.1, D1.C, D8.C, IC2.VI, K42.S, K72.S, R14.1, R24.1
- net HIGH_TEMPERATURE_1: now also R14.2, R28.1, R38.1; no longer R29.2, R34.1
- net HIGH_TEMPERATURE_2: now also R23.2, R29.1, R37.1; no longer R25.2, R26.1
- net N$1: now also K22.P, R8.2; no longer K42.P, R14.2
- net N$12: now also D9.C, K41.1, K61.1, Q5.C, R32.1; no longer D7.C, K21.1, K31.1, Q3.C, R13.1
- net N$13: now also R32.2; no longer R13.2
- net N$14: now also R26.1; no longer R12.1
- net N$15: now also C9.+, D4.A, D5.C, R12.E; no longer C7.+, D1.A, D2.C, R3.E
- net N$16: now also C8.+, D5.A, R12.A, R12.S, R13.E; no longer C6.+, D2.A, R3.A, R3.S, R4.E
- net N$17: now also K32.O; no longer K12.O
- net N$18: now also R3.1, R4.2; no longer R20.1, R21.2
- net N$19: now also R35.1; no longer D3.A
- net N$2: now also D1.A, K11.2, K21.2; no longer D6.A, K41.2, K71.2
- net N$20: now also R36.1; no longer D4.A
- net N$21: now also R21.1, R22.2, R24.1; no longer R10.1, R8.1, R9.2
- net N$22: now also R16.2; no longer R5.2
- net N$25: now also R7.S; no longer R2.S
- net N$26: now also C13.+, D6.A, D7.C, R30.E; no longer C11.+, D5.C, D8.A, R23.E
- net N$27: now also C12.+, D7.A, R30.A, R30.S, R31.E; no longer C10.+, D5.A, R22.E, R23.A, R23.S
- net N$29: now also K12.P, R25.2; no longer K72.P, R24.2
- net N$3: now also R27.1; no longer R11.1
- net N$30: now also R15.S, R23.1; no longer R25.1, R33.S
- net N$31: now also R19.1, R20.E, R20.S; no longer R27.1, R32.E, R32.S
- net N$34: now also R29.2; no longer R26.2
- net N$35: now also R10.1, R11.E, R11.S; no longer R28.1, R30.E, R30.S
- net N$36: now also R14.1, R9.S; no longer R29.1, R31.S
- net N$38: now also D8.C, L1.1, Q3.C; no longer D10.C, L2.1, Q5.C
- net N$4: now also R6.2; no longer R15.2
- net N$5: now also R5.2, R6.1; no longer R15.1, R18.2
- net N$6: now also R1.S; no longer R19.S
- net SHORT_CIRCUIT_MONITOR_1: now also K32.P; no longer K12.P
Other:
- note added: "1.1"
- note added: "VREF = 6.00V at 21°C"
- note added: "VREF = 8.00V"
- note removed: "1.0"
- moved on the sheet: C10, C2, C3, C6, C8, D1, D4, D5, D6, D7, D8, IC1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

Commit message: Minor improvements
Parts:
- removed K5: APF30212C, relay:APF30212C
- removed K6: 12VDC, relay:APF30212C
- removed KK1, KK2: D0A-L, heatsink:D0A-L
- removed LD1: Bicolor AC (Red/Green), led:DUOLED-RG-A
- removed R35, R36: 1k (5%), rcl:R-EU_0207/7
- removed R37, R38: 10k (5%), rcl:R-EU_0207/7
- removed SW1: CT10-XXXX-A2, switch-coto:CT10-XXXX-A2
- removed T1: BC337, transistor-neu-to92:BC337
- added C14, C15: 10uF x 50V, rcl:CPOL-EU153CLV-0605
- added D2, D3: 1N4007, diode:CGRM4007-G
- added LED1: Bicolor LED Common-Anode, led:LED-BICOLOR-MOLEX3P
- added Q6: BC858BSMD, transistor-pnp:BC858BSMD
- added RT1, RT4: 5R, ptc-ntc:NTC-11MM
- added RT2, RT3: 10k, ptc-ntc:NTC-MOLEX2P
- added S2: SWITCH-MOLEX2P, switch-MOLEX2:SWITCH-MOLEX2P
- C1, C2: device rcl:C-EU025-025X050 -> rcl:C-EUC0805
- C10: value 15.000uF x 50V -> (none); device rcl:CPOL-EUE10-35 -> rcl:C-EUC0805
- C11, C4: value 100nF x 50V -> 10uF x 50V; device rcl:C-EU025-025X050 -> rcl:CPOL-EU153CLV-0605
- C12: value 10uF x 50V -> 15.000uF x 50V; device rcl:CPOL-EUE3.5-8 -> rcl:CPOL-EUE10-35
- C13, C3, C5, C8: value 10uF x 50V -> 100nF x 50V; device rcl:CPOL-EUE3.5-8 -> rcl:C-EUC0805
- C6: value 15.000uF x 50V -> 10uF x 50V; device rcl:CPOL-EUE10-35 -> rcl:CPOL-EU153CLV-0605
- C7: value 100nF x 50V -> 15.000uF x 50V; device rcl:C-EU025-025X050 -> rcl:CPOL-EUE10-35
- C9: device rcl:CPOL-EUE3.5-8 -> rcl:CPOL-EU153CLV-0605
- D1, D6, D7: value 1N4007 -> 1N4148; device diode:1N5060GP -> diode:DIODE-SOD523
- D4, D5, D8, D9: device diode:1N5060GP -> diode:CGRM4007-G
- F1: value (none) -> FUSE; device fuse:19559 -> fuse-no-footprint:FUSE
- IC3: value LM324N -> LM324D; device linear:LM324N -> linear:LM324D
- IC4: value LM358N -> LM358D; device linear:LM358N -> linear:LM358D
- K1, K2, K4: value 12VDC -> 12VDC COIL; device relay:APF30212C -> relay:ZNS5448
- K3: value APF30212C -> 12VDC COIL; device relay:APF30212C -> relay:ZNS5448
- L1: value Cooler 24V @ 6W -> MOTOR; device Inductor:INDUCTOR -> Inductor:MOTOR
- Q1: value BC548B -> BC848SMD; device transistor-npn:BC548B -> transistor-npn:BC848SMD
- Q2: value BC558B -> BC848BSMD; device transistor-pnp:BC558B -> transistor-npn:BC848BSMD
- Q3, Q4, Q5: value BC558B -> BC858BSMD; device transistor-pnp:BC558B -> transistor-pnp:BC858BSMD
- R10: value 10k -> 1k (5%); device ptc-ntc:NTC640 -> rcl:R-EU_R0805
- R11: value 10k -> 1k (5%); device rcl:R-TRIMM64W -> rcl:R-EU_R0805
- R12: value 500R -> 33k (5%); device rcl:R-TRIMMT93YB -> rcl:R-EU_R0805
- R13: value 5K -> 500R; device pot:3RP/1610N -> rcl:R-TRIMM64W
- R14: value 33k (5%) -> 5K; device rcl:R-EU_0207/7 -> trimpot-molex2p:R-TRIMM
- R16, R18, R21, R28, R3, R33, R34, R4, R5, R6: device rcl:R-EU_0207/7 -> rcl:R-EU_R0805
- R17: value 100k (1%) -> 10k; device rcl:R-EU_0207/7 -> rcl:R-TRIMM64W
- R19: value 10k -> 100k (1%); device ptc-ntc:NTC640 -> rcl:R-EU_R0805
- R2: value VARISTOR-2,5 -> VARISTOR; device varistor:VARISTOR-2,5 -> varistor:VARISTOR
- R20: value 10k -> 100k (1%); device rcl:R-TRIMM64W -> rcl:R-EU_R0805
- R22: value 100k (1%) -> 33k (5%); device rcl:R-EU_0207/7 -> rcl:R-EU_R0805
- R23: value 33k (5%) -> 220k (5%); device rcl:R-EU_0207/7 -> rcl:R-EU_R0805
- R24: value 220k (5%) -> 10k (5%); device rcl:R-EU_0207/7 -> rcl:R-EU_R0805
- R25: value 5R -> 1k (5%); device ptc-ntc:NTC640 -> rcl:R-EU_R0805
- R26: value 10k (5%) -> 500R; device rcl:R-EU_0207/7 -> rcl:R-TRIMM64W
- R27: value 1k (5%) -> 5K; device rcl:R-EU_0207/7 -> trimpot-molex2p:R-TRIMM
- R29: value 10k (5%) -> 1k (5%); device rcl:R-EU_0207/7 -> rcl:R-EU_R0805
- R30: value 500R -> 10k (5%); device rcl:R-TRIMMT93YB -> rcl:R-EU_R0805
- R31: value 5K -> 10k (5%); device pot:3RP/1610N -> rcl:R-EU_R0805
- R32: value 1k (5%) -> 10k (5%); device rcl:R-EU_0207/7 -> rcl:R-EU_R0805
- R8: value 5R -> 10k; device ptc-ntc:NTC640 -> rcl:R-TRIMM64W
- S1: device switch:320-938 -> switch-HH-NO-MODEL:320-938
- TR1, TR2: value 24V @ 5A -> TRAFO
- U1, U2: device REG1117:REG1117F -> REG1117:LM338K-MOLEX
- X1, X2: value (none) -> 22-23-2021; device con-ptr500:AK500/4-H -> con-molex-PTR:22-23-2021
- renumbered TR?1 to TR1, TR?2 to TR2
Connections:
- new net 30V_A: C7.+, C8.1, D2.C, D8.A, K22.S, RT1.1, U1.VIN
- new net 30V_B: C12.+, C13.1, D4.C, D9.A, K12.S, RT4.1, U2.VIN
- net !SHORT_CIRCUIT_DETECTED!: now also Q2.C, R10.2, R11.2; no longer Q1.C, R35.2, R36.2
- net !VOUT1_POWER_OFF!: now also R23.2, R25.2; no longer R24.2, R27.2
- net !VOUT1_POWER_ON!: now also R18.1, R19.2, R24.2, S2.2; no longer R17.1, R18.2, R26.2, SW1.2
- net +24V: now also C10.1, C3.1, C4.+, Q5.E, R28.2, R30.2, R8.E, RT2.2, RT3.2, VOLT1.P$1, VOLT2.P$1; no longer C3.+, Q3.E, R10.2, R19.2, R37.2, R38.2, R9.E
- net 0V: now also C10.2, C11.-, C13.2, C14.-, C15.-, C3.2, C4.-, C5.2, C7.-, C8.2, D6.A, D7.A, K31.2, Q1.E, Q3.C, R14.A, R14.S, R17.A, R19.1, R21.1, R27.A, R27.S, R8.A, S2.1, X1-2.S, X2-2.S; no longer C10.-, C11.2, C13.-, C3.-, C4.2, C5.-, C7.2, C8.-, D8.A, D9.A, K61.2, Q2.C, R11.A, R13.A, R13.S, R18.1, R20.A, R22.1, R31.A, R31.S, SW1.1, T1.E, X1-2.KL, X2-2.KL
- net 0V_A: no longer TR1.GRN/YEL1, TR2.GRN/YEL1
- net 0V_B: no longer TR1.GRN/YEL, TR2.GRN/YEL
- net 127V_A: no longer TR1.BLK@1, TR2.BLK@1
- net 127V_B: no longer TR1.BLK@2, TR2.BLK@2
- net 12V: now also C5.1, C6.+, LED1.A, Q6.E, R18.2, R20.2; no longer C4.1, C5.+, LD1.A, Q5.E, R17.2, R21.2
- net 30V: now also D8.C, D9.C; no longer C10.+, C11.1, C6.+, C7.1, D4.C, D6.C, K12.S, K22.S, R25.1, R8.1, U1.VIN, U2.VIN
- net HIGH_TEMPERATURE_1: now also R12.2, R31.1; no longer R14.2, R38.1
- net HIGH_TEMPERATURE_2: now also R22.2, R30.1, R32.1; no longer R23.2, R29.1, R37.1
- net N$1: now also RT1.2; no longer R8.2
- net N$10: now also TR1.1; no longer TR1.GRN@1
- net N$11: now also TR1.2; no longer TR1.GRN@2
- net N$12: now also D7.C, K31.1, Q3.E, Q6.C, R29.1; no longer D9.C, K61.1, Q2.E, Q5.C, R32.1
- net N$13: now also LED1.CG, R29.2; no longer LD1.CG, R32.2
- net N$14: now also Q3.B, R24.1; no longer Q2.B, R26.1
- net N$15: now also C11.+, D2.A, D3.C, R13.E; no longer C9.+, D4.A, D5.C, R12.E
- net N$16: now also C9.+, D3.A, R13.A, R13.S, R14.E; no longer C8.+, D5.A, R12.A, R12.S, R13.E
- net N$17: now also K42.O, X1-1.S; no longer K32.O, X1-1.KL
- net N$19: now also R10.1; no longer R35.1
- net N$2: now also Q1.C; no longer T1.C
- net N$20: now also R11.1; no longer R36.1
- net N$21: now also Q2.E, R20.1, R21.2, R23.1; no longer Q1.E, R21.1, R22.2, R24.1
- net N$22: now also Q2.B; no longer Q1.B
- net N$23: now also TR2.1; no longer TR2.GRN@1
- net N$24: now also TR2.2; no longer TR2.GRN@2
- net N$26: now also C15.+, D4.A, D5.C, R26.E; no longer C13.+, D6.A, D7.C, R30.E
- net N$27: now also C14.+, D5.A, R26.A, R26.S, R27.E; no longer C12.+, D7.A, R30.A, R30.S, R31.E
- net N$28: now also K32.O, X2-1.S; no longer K52.O, X2-1.KL
- net N$29: now also RT4.2; no longer R25.2
- net N$3: now also LED1.CR, R25.1; no longer LD1.CR, R27.1
- net N$30: now also R22.1; no longer R23.1
- net N$31: now also R17.E, R17.S, RT3.1; no longer R19.1, R20.E, R20.S
- net N$32: now also Q4.B, R31.2; no longer Q3.B, R28.2
- net N$34: now also Q5.B, R32.2; no longer Q4.B, R29.2
- net N$35: now also R9.E, R9.S, RT2.1; no longer R10.1, R11.E, R11.S
- net N$36: now also R12.1, R8.S; no longer R14.1, R9.S
- net N$38: now also D6.C, Q5.C; no longer D8.C, Q3.C
- net N$4: now also Q1.B; no longer T1.B
- net N$7: now also Q6.B; no longer Q5.B
- net SHORT_CIRCUIT_MONITOR_1: now also K42.P; no longer K52.P
Other:
- note added: "1"
- note added: "2"
- note added: "3"
- note added: "4"
- note added: "5"
- note added: "6"
- moved on the sheet: C12, C2, C6, C9, IC4A, IC4B, K1, K2, K3, K4, Q1, Q3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

Commit message: PCB layout done
Parts:
- added C16: 100nF x 50V, rcl:C-EUC0805
Connections:
- net +24V: now also C16.1
- net 0V: now also C16.2
- net SHORT_CIRCUIT_MONITOR_1: no longer AMP2.P$2, K32.P, VOLT2.P$3
- net SHORT_CIRCUIT_MONITOR_2: now also AMP2.P$2, K32.P, VOLT2.P$3
Other:
- moved on the sheet: C3, C4
Changed lines of the file:
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@@
 <setting verticaltext="up"/>
 </settings>
-<grid distance="25" unitdist="mil" unit="mil" style="lines" multiple="1" display="no" altdistance="0.01" altunitdist="inch" altunit="inch"/>
+<grid distance="0.1" unitdist="inch" unit="inch" style="lines" multiple="1" display="no" altdistance="0.01" altunitdist="inch" altunit="inch"/>
 <layers>
 <layer number="1" name="Top" color="4" fill="1" visible="no" active="no"/>
@@
 <part name="D8" library="diode" library_urn="urn:adsk.eagle:library:210" deviceset="CGRM400*-G" device="" package3d_urn="urn:adsk.eagle:package:43457/2" technology="7" value="1N4007"/>
 <part name="D9" library="diode" library_urn="urn:adsk.eagle:library:210" deviceset="CGRM400*-G" device="" package3d_urn="urn:adsk.eagle:package:43457/2" technology="7" value="1N4007"/>
+<part name="C16" library="rcl" library_urn="urn:adsk.eagle:library:334" deviceset="C-EU" device="C0805" package3d_urn="urn:adsk.eagle:package:23617/2" value="100nF x 50V"/>
+<part name="GND30" library="supply1" library_urn="urn:adsk.eagle:library:371" deviceset="0V" device=""/>
 </parts>
 <sheets>
@@
 <attribute name="VALUE" x="10.795" y="85.09" size="1.778" layer="96"/>
 </instance>
-<instance part="C3" gate="G$1" x="47.625" y="36.195" smashed="yes">
-<attribute name="NAME" x="40.894" y="34.036" size="1.778" layer="95"/>
-<attribute name="VALUE" x="52.324" y="28.829" size="1.778" layer="96" rot="R90"/>
+<instance part="C3" gate="G$1" x="42.545" y="36.195" smashed="yes">
+<attribute name="NAME" x="38.354" y="39.116" size="1.778" layer="95"/>
+<attribute name="VALUE" x="47.244" y="28.829" size="1.778" layer="96" rot="R90"/>
 </instance>
 <instance part="C1" gate="G$1" x="12.7" y="36.195" smashed="yes">
@@
 <attribute name="VALUE" x="17.399" y="28.194" size="1.778" layer="96" rot="R90"/>
 </instance>
-<instance part="C4" gate="G$1" x="61.595" y="36.195" smashed="yes">
-<attribute name="NAME" x="55.118" y="34.1376" size="1.778" layer="95"/>
-<attribute name="VALUE" x="66.1924" y="29.718" size="1.778" layer="96" rot="R90"/>
+<instance part="C4" gate="G$1" x="53.975" y="36.195" smashed="yes">
+<attribute name="NAME" x="50.038" y="39.2176" size="1.778" layer="95"/>
+<attribute name="VALUE" x="58.5724" y="29.718" size="1.778" layer="96" rot="R90"/>
 </instance>
 <instance part="GND2" gate="1" x="12.7" y="18.415" smashed="yes">
 <attribute name="VALUE" x="11.43" y="15.875" size="1.778" layer="96"/>
 </instance>
-<instance part="GND8" gate="1" x="47.625" y="18.415" smashed="yes">
-<attribute name="VALUE" x="46.355" y="15.875" size="1.778" layer="96"/>
-</instance>
-<instance part="GND9" gate="1" x="61.595" y="18.415" smashed="yes">
-<attribute name="VALUE" x="60.325" y="15.875" size="1.778" layer="96"/>
-</instance>
-<instance part="SUPPLY5" gate="+24V" x="61.595" y="81.915" smashed="yes">
-<attribute name="VALUE" x="59.69" y="85.09" size="1.778" layer="96"/>
+<instance part="GND8" gate="1" x="42.545" y="18.415" smashed="yes">
+<attribute name="VALUE" x="41.275" y="15.875" size="1.778" layer="96"/>
+</instance>
+<instance part="GND9" gate="1" x="53.975" y="18.415" smashed="yes">
+<attribute name="VALUE" x="52.705" y="15.875" size="1.778" layer="96"/>
+</instance>
+<instance part="SUPPLY5" gate="+24V" x="53.975" y="81.915" smashed="yes">
+<attribute name="VALUE" x="52.07" y="85.09" size="1.778" layer="96"/>
 </instance>
 <instance part="IC4" gate="A" x="167.005" y="52.705" smashed="yes">
@@
 <attribute name="NAME" x="301.7774" y="233.045" size="1.27" layer="95" rot="MR270"/>
 <attribute name="VALUE" x="299.4914" y="234.95" size="1.27" layer="96" rot="MR270"/>
+</instance>
+<instance part="C16" gate="G$1" x="65.405" y="36.195" smashed="yes">
+<attribute name="NAME" x="60.579" y="39.116" size="1.778" layer="95"/>
+<attribute name="VALUE" x="70.104" y="28.829" size="1.778" layer="96" rot="R90"/>
+</instance>
+<instance part="GND30" gate="1" x="65.405" y="18.415" smashed="yes">
+<attribute name="VALUE" x="64.135" y="15.875" size="1.778" layer="96"/>
 </instance>
 </instances>
@@
 <pinref part="C3" gate="G$1" pin="2"/>
 <pinref part="GND8" gate="1" pin="0V"/>
-<wire x1="47.625" y1="31.115" x2="47.625" y2="20.955" width="0.1524" layer="91"/>
+<wire x1="42.545" y1="31.115" x2="42.545" y2="20.955" width="0.1524" layer="91"/>
 </segment>
 <segment>
 <pinref part="C4" gate="G$1" pin="-"/>
 <pinref part="GND9" gate="1" pin="0V"/>
-<wire x1="61.595" y1="31.115" x2="61.595" y2="20.955" width="0.1524" layer="91"/>
+<wire x1="53.975" y1="31.115" x2="53.975" y2="20.955" width="0.1524" layer="91"/>
 </segment>
 <segment>
@@
 <wire x1="183.515" y1="69.215" x2="183.515" y2="69.85" width="0.1524" layer="91"/>
 </segment>
+<segment>
+<pinref part="C16" gate="G$1" pin="2"/>
+<pinref part="GND30" gate="1" pin="0V"/>
+<wire x1="65.405" y1="31.115" x2="65.405" y2="20.955" width="0.1524" layer="91"/>
+</segment>
 </net>
 <net name="SHORT_CIRCUIT_MONITOR_1" class="0">
@@
 <pinref part="AMP1" gate="G$1" pin="P$2"/>
 <pinref part="VOLT1" gate="G$1" pin="P$3"/>
-</segment>
-<segment>
-<wire x1="375.92" y1="215.9" x2="375.92" y2="227.33" width="0.1524" layer="91"/>
-<wire x1="375.92" y1="227.33" x2="372.11" y2="227.33" width="0.1524" layer="91"/>
-<wire x1="375.92" y1="234.95" x2="375.92" y2="227.33" width="0.1524" layer="91"/>
-<junction x="375.92" y="227.33"/>
-<label x="386.715" y="227.33" size="1.27" layer="95" rot="R270" xref="yes"/>
-<wire x1="375.92" y1="227.33" x2="386.715" y2="227.33" width="0.1524" layer="91"/>
-<pinref part="K3" gate="2" pin="P"/>
-<pinref part="AMP2" gate="G$1" pin="P$2"/>
-<pinref part="VOLT2" gate="G$1" pin="P$3"/>
 </segment>
 </net>
@@
 <segment>
 <pinref part="C4" gate="G$1" pin="+"/>
-<wire x1="61.595" y1="38.735" x2="61.595" y2="51.435" width="0.1524" layer="91"/>
-<wire x1="39.37" y1="51.435" x2="47.625" y2="51.435" width="0.1524" layer="91"/>
-<wire x1="47.625" y1="51.435" x2="61.595" y2="51.435" width="0.1524" layer="91"/>
+<wire x1="53.975" y1="38.735" x2="53.975" y2="51.435" width="0.1524" layer="91"/>
+<wire x1="39.37" y1="51.435" x2="42.545" y2="51.435" width="0.1524" layer="91"/>
+<wire x1="42.545" y1="51.435" x2="53.975" y2="51.435" width="0.1524" layer="91"/>
 <pinref part="C3" gate="G$1" pin="1"/>
-<wire x1="47.625" y1="38.735" x2="47.625" y2="51.435" width="0.1524" layer="91"/>
-<junction x="47.625" y="51.435"/>
+<wire x1="42.545" y1="38.735" x2="42.545" y2="51.435" width="0.1524" layer="91"/>
+<junction x="42.545" y="51.435"/>
 <pinref part="IC1" gate="A1" pin="VO"/>
 <pinref part="SUPPLY5" gate="+24V" pin="+24V"/>
-<wire x1="61.595" y1="79.375" x2="61.595" y2="51.435" width="0.1524" layer="91"/>
-<junction x="61.595" y="51.435"/>
+<wire x1="53.975" y1="79.375" x2="53.975" y2="51.435" width="0.1524" layer="91"/>
+<junction x="53.975" y="51.435"/>
 <pinref part="IC2" gate="A1" pin="VI"/>
-<wire x1="61.595" y1="51.435" x2="69.85" y2="51.435" width="0.1524" layer="91"/>
+<wire x1="53.975" y1="51.435" x2="65.405" y2="51.435" width="0.1524" layer="91"/>
+<wire x1="65.405" y1="51.435" x2="69.85" y2="51.435" width="0.1524" layer="91"/>
+<wire x1="62.23" y1="51.435" x2="65.405" y2="51.435" width="0.1524" layer="91"/>
+<pinref part="C16" gate="G$1" pin="1"/>
+<wire x1="65.405" y1="38.735" x2="65.405" y2="51.435" width="0.1524" layer="91"/>
+<junction x="65.405" y="51.435"/>
 </segment>
 <segment>
@@
 <label x="120.65" y="138.43" size="1.27" layer="95" ratio="5" rot="R180" xref="yes"/>
 </segment>
-</net>
+<segment>
+<wire x1="375.92" y1="215.9" x2="375.92" y2="227.33" width="0.1524" layer="91"/>
+<wire x1="375.92" y1="227.33" x2="372.11" y2="227.33" width="0.1524" layer="91"/>
+<wire x1="375.92" y1="234.95" x2="375.92" y2="227.33" width="0.1524" layer="91"/>
+<junction x="375.92" y="227.33"/>
+<label x="386.715" y="227.33" size="1.27" layer="95" rot="R270" xref="yes"/>
+<wire x1="375.92" y1="227.33" x2="386.715" y2="227.33" width="0.1524" layer="91"/>
+<pinref part="K3" gate="2" pin="P"/>
+<pinref part="AMP2" gate="G$1" pin="P$2"/>
+<pinref part="VOLT2" gate="G$1" pin="P$3"/>
+</segment>
+</net>
