File: Hardware/0. Project/AC-DC.sch (EAGLE design)
At the start: 95 parts, among them IC1 7824TV, IC2 7812TV, IC3 LM324D, IC4 LM358D, K1 12VDC COIL, K2 12VDC COIL, K3 12VDC COIL, K4 12VDC COIL, Q1 BC848SMD, Q2 BC848BSMD, Q3 BC858BSMD, Q4 BC858BSMD, Q5 BC858BSMD, Q6 BC858BSMD, U1 LM338K, U2 LM338K, X1 22-23-2021, X2 22-23-2021

Commit message: Schematic updated to 2.0
- All Op. Amps. that was voltage compators was updated to LM393.
- Fixed conflicts at +12V and +24V lines.
- Now, there is only one temperature circuit monitor.
- Ground from supply1 and supply2 is now isolated from each other
(series and parallel association are now possible).
Parts:
- removed C1, C16, C2, C3: 100nF x 50V, rcl:C-EUC0805
- removed C10: (no value), rcl:C-EUC0805
- removed C4: 10uF x 50V, rcl:CPOL-EU153CLV-0605
- removed IC1: 7824TV, linear:7824TV
- removed IC2: 7812TV, linear:7812TV
- removed IC3: LM324D, linear:LM324D
- removed Q5: BC858BSMD, transistor-pnp:BC858BSMD
- removed R15, R17: 10k, rcl:R-TRIMM64W
- removed R22: 33k (5%), rcl:R-EU_R0805
- removed R30, R32: 10k (5%), rcl:R-EU_R0805
- removed RT3: 10k, ptc-ntc:NTC-MOLEX2P
- added D10: (no value), diode:ZENER-DIODESOD80C
- added IC5, IC6: LM393D, linear:LM393D
- added OK1, OK2, OK3, OK4: 4N33, optocoupler:4N33
- added Q7: BC848SMD, transistor-npn:BC848SMD
- added R35, R38, R46, R49: 100k (5%), rcl:R-EU_R0805
- added R36, R44, R48: 1k (5%), rcl:R-EU_R0805
- added R37, R39, R43, R47: 10k (5%), rcl:R-EU_R0805
- added R40: 500k, rcl:R-TRIMM64W
- added R41: 100k (1%), rcl:R-EU_R0805
- added R42: 33k (1%), rcl:R-EU_R0805
- added R45, R50: (no value), rcl:R-EU_R2512
- added U3: HLK-PM01, HLK-PM01:HLK-PM01
- D8: value 1N4007 -> 1N4148; device diode:CGRM4007-G -> diode:DIODE-SOD523
- D9: value 1N4007 -> (none); device diode:CGRM4007-G -> diode:ZENER-DIODESOD80C
- R10: value 1k (5%) -> 10k (5%)
- R5: value 10k (5%) -> 500k; device rcl:R-EU_R0805 -> rcl:R-TRIMM64W
- TR1, TR2: value TRAFO -> 24VRMS
Connections:
- removed net 0V: B1.-, B2.-, C1.2, C10.2, C11.-, C12.-, C13.2, C14.-, C15.-, C16.2, C2.2, C3.2, C4.-, C5.2, C6.-, C7.-, C8.2, C9.-, D6.A, D7.A, IC1.GND, IC2.GND, IC3P.V-, IC4P.V-, K31.2, K41.2, L1.2, Q1.E, Q3.C, R1.A, R14.A, R14.S, R15.A, R17.A, R19.1, R21.1, R27.A, R27.S, R33.2, R4.1, R5.1, R7.A, R8.A, R9.A, S2.1, VOLT1.P$2, VOLT2.P$2, X1-2.S, X2-2.S
- removed net 12V: C5.1, C6.+, IC2.VO, LED1.A, Q6.E, R18.2, R20.2, R7.E
- removed net 30V: C1.1, D8.C, D9.C, IC1.VI
- removed net 30V_A: C7.+, C8.1, D2.C, D8.A, K22.S, RT1.1, U1.VIN
- removed net 30V_B: C12.+, C13.1, D4.C, D9.A, K12.S, RT4.1, U2.VIN
- removed net HIGH_TEMPERATURE_2: IC4B.OUT, R22.2, R30.1, R32.1
- removed net N$30: IC4B.+IN, R15.S, R22.1
- removed net N$31: IC4B.-IN, R17.E, R17.S, RT3.1
- removed net N$34: Q5.B, R32.2
- removed net SHORT_CIRCUIT_MONITOR_1: AMP1.P$2, IC3A.+IN, K42.P, VOLT1.P$3
- removed net SHORT_CIRCUIT_MONITOR_2: AMP2.P$2, IC3D.+IN, K32.P, VOLT2.P$3
- new net !VOUT1_POWER_ON!1: OK1.COL, R11.1
- new net !VOUT1_POWER_ON!2: OK2.COL, R36.1
- new net !VOUT1_POWER_ON!3: OK3.COL, R44.1
- new net !VOUT1_POWER_ON!4: OK4.COL, R48.1
- new net +12V: C5.1, C6.+, D1.C, D8.C, IC4P.V+, K11.1, K21.1, LED1.A, Q4.E, Q6.E, R11.2, R18.2, R20.2, R28.2, R36.2, R44.2, R48.2, R8.E, RT2.2, U3.VO+
- new net 12V_AUX1: D9.C, IC5P.V+, R1.E, R45.1, R7.E
- new net 12V_AUX2: D10.C, IC6P.V+, R40.E, R5.E, R50.1
- new net C_FULL_1: C7.+, C8.1, D2.C, K22.S, R3.2, R45.2, RT1.1, U1.VIN
- new net C_FULL_2: C12.+, C13.1, D4.C, K12.S, R41.2, R50.2, RT4.1, U2.VIN
- new net GND1: B1.-, C11.-, C7.-, C8.2, C9.-, D9.A, IC5P.V-, OK1.C, OK2.C, R1.A, R14.A, R14.S, R33.2, R4.1, R7.A, VOLT1.P$2, X1-2.S
- new net GND2: B2.-, C12.-, C13.2, C14.-, C15.-, D10.A, IC6P.V-, OK3.C, OK4.C, R27.A, R27.S, R40.A, R42.1, R5.A, VOLT2.P$2, X2-2.S
- new net HIGH_TEMPERATURE: IC4A.OUT, R12.2
- new net N$33: D8.A, K11.2, Q7.C
- new net N$37: IC5B.OUT, R37.1
- new net N$39: OK2.A, R37.2
- new net N$40: Q7.B, R39.2
- new net N$41: IC6B.+IN, R41.1, R42.2
- new net N$42: IC6A.OUT, R43.1
- new net N$43: IC6B.-IN, R40.S
- new net N$44: OK3.A, R43.2
- new net N$45: IC6B.OUT, R47.1
- new net N$46: OK4.A, R47.2
- new net N$47: OK4.E, R39.1, R49.2
- new net N$48: OK2.E, R38.2, R6.1
- new net PE: C5.2, C6.-, D6.A, D7.A, IC4P.V-, K31.2, K41.2, L1.2, Q1.E, Q3.C, Q7.E, R19.1, R21.1, R35.1, R38.1, R46.1, R49.1, R8.A, R9.A, S2.1, U3.VO-
- new net VOUT_1: AMP1.P$2, IC5A.+IN, IC6A.+IN, K42.P, VOLT1.P$3
- new net VOUT_2: AMP2.P$2, K32.P, VOLT2.P$3
- net !SHORT_CIRCUIT_DETECTED!: now also OK1.E, OK3.E, R35.2, R46.2; no longer R10.2, R11.2
- net !VOUT1_POWER_OFF!: now also IC4B.OUT; no longer IC3B.OUT
- net !VOUT1_POWER_ON!: now also IC4B.-IN; no longer IC3B.-IN
- net +24V: no longer C10.1, C16.1, C2.1, C3.1, C4.+, D1.C, IC1.VO, IC2.VI, IC3P.V+, IC4P.V+, K11.1, K21.1, Q4.E, Q5.E, R1.E, R15.E, R28.2, R3.2, R30.2, R8.E, RT2.2, RT3.2
- net 0V_B: now also U3.AC2
- net 127V_B: now also U3.AC1
- net HIGH_TEMPERATURE_1: no longer IC4A.OUT, R12.2
- net N$18: now also IC5B.+IN; no longer IC3C.+IN
- net N$19: now also IC5A.OUT; no longer IC3A.OUT
- net N$2: no longer K11.2
- net N$20: now also OK1.A, R10.2; no longer IC3D.OUT, R11.1
- net N$21: now also IC4B.+IN; no longer IC3B.+IN
- net N$25: now also IC5A.-IN; no longer IC3A.-IN, IC3D.-IN
- net N$38: no longer Q5.C
- net N$5: now also IC6A.-IN, R5.S; no longer IC3C.OUT, R5.2, R6.1
- net N$6: now also IC5B.-IN; no longer IC3C.-IN
Other:
- note added: "2.0"
- note added: "3W / 12V"
- note added: "TEMPERATURE MONITOR HEAT SINK"
- note removed: "1.1"
- note removed: "TEMPERATURE MONITOR VOLTAGE REGULATOR 1"
- note removed: "TEMPERATURE MONITOR VOLTAGE REGULATOR 2"
- moved on the sheet: B1, B2, C11, C12, C13, C14, C15, C5, C6, C7, C8, C9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

Commit message: Schematic 2.0 done
Parts:
- removed C12: 15.000uF x 50V, rcl:CPOL-EUE10-35
- removed C13: 100nF x 50V, rcl:C-EUC0805
- removed C14: 10uF x 50V, rcl:CPOL-EU153CLV-0605
- removed IC4: LM358D, linear:LM358D
- removed Q7: BC848SMD, transistor-npn:BC848SMD
- removed R46, R49: 100k (5%), rcl:R-EU_R0805
- removed R47: 10k (5%), rcl:R-EU_R0805
- removed R48: 1k (5%), rcl:R-EU_R0805
- removed R50: (no value), rcl:R-EU_R2512
- removed RT4: 5R, ptc-ntc:NTC-11MM
- added C1: 15.000uF x 50V, rcl:CPOL-EUE10-35
- added C2: 100nF x 50V, rcl:C-EUC0805
- added C3: 10uF x 50V, rcl:CPOL-EU153CLV-0605
- added IC3: LM358D, linear:LM358D
- added Q5: BC858, transistor-pnp:BC858BSMD
- added R15, R32: 10k (5%), rcl:R-EU_R0805
- added R17: 500k, rcl:R-TRIMM64W
- added R22: 220R, rcl:R-EU_R2512
- added R30: 1k (5%), rcl:R-EU_R0805
- added RT3: 10k, ptc-ntc:NTC-MOLEX2P
- D1: value 1N4148 -> 12V / 0.5W; device diode:DIODE-SOD523 -> diode:ZENER-DIODESOD80C
- D10, D9: value (none) -> 1N4148; device diode:ZENER-DIODESOD80C -> diode:DIODE-SOD523
- D4: value 1N4007 -> 1N4148; device diode:CGRM4007-G -> diode:DIODE-SOD523
- D5: value 1N4007 -> 12V / 0.5W; device diode:CGRM4007-G -> diode:ZENER-DIODESOD80C
- D6, D7: value 1N4148 -> 1N4007; device diode:DIODE-SOD523 -> diode:CGRM4007-G
- Q1: value BC848SMD -> BC848
- Q2: value BC848BSMD -> BC848; device transistor-npn:BC848BSMD -> transistor-npn:BC848SMD
- Q3, Q6: value BC858BSMD -> BC858
- Q4: value BC858BSMD -> BC848; device transistor-pnp:BC858BSMD -> transistor-npn:BC848BSMD
- R10: value 10k (5%) -> 5K; device rcl:R-EU_R0805 -> trimpot-molex2p:R-TRIMM
- R12: value 33k (5%) -> 100k (5%)
- R13: value 500R -> 1k (5%); device rcl:R-TRIMM64W -> rcl:R-EU_R0805
- R14: value 5K -> 100k (5%); device trimpot-molex2p:R-TRIMM -> rcl:R-EU_R0805
- R16: value 10k (5%) -> 500k; device rcl:R-EU_R0805 -> rcl:R-TRIMM64W
- R19, R21: value 100k (1%) -> 10k; device rcl:R-EU_R0805 -> rcl:R-TRIMM64W
- R2: value VARISTOR -> 500k; device varistor:VARISTOR -> rcl:R-TRIMM64W
- R20: value 100k (1%) -> 33k (1%)
- R23: value 220k (5%) -> 10k (5%)
- R25: value 1k (5%) -> 33k (5%)
- R28, R34: value 10k (5%) -> 1k (5%)
- R29, R44: value 1k (5%) -> 100k (5%)
- R3: value 100k (1%) -> VARISTOR; device rcl:R-EU_R0805 -> varistor:VARISTOR
- R31: value 10k (5%) -> 100k (5%)
- R33, R35: value 100k (5%) -> 10k (5%)
- R37: value 10k (5%) -> 100k (1%)
- R38: value 100k (5%) -> 100k (1%)
- R4: value 33k (1%) -> 100k (1%)
- R40: value 500k -> 100k (1%); device rcl:R-TRIMM64W -> rcl:R-EU_R0805
- R42: value 33k (1%) -> 10k (5%)
- R43: value 10k (5%) -> 220k (5%)
- R45: value (none) -> 10k (5%); device rcl:R-EU_R2512 -> rcl:R-EU_R0805
- R5: value 500k -> 33k (1%); device rcl:R-TRIMM64W -> rcl:R-EU_R0805
- R6: value 10k (5%) -> 220R; device rcl:R-EU_R0805 -> rcl:R-EU_R2512
- R7: value 500k -> 10k (5%); device rcl:R-TRIMM64W -> rcl:R-EU_R0805
- R8: value 10k -> 10k (5%); device rcl:R-TRIMM64W -> rcl:R-EU_R0805
- R9: value 10k -> 500R
- RT2: value 10k -> 5R; device ptc-ntc:NTC-MOLEX2P -> ptc-ntc:NTC-11MM
- U2: value LM338K -> HLK-PM01; device REG1117:LM338K-MOLEX -> HLK-PM01:HLK-PM01
- U3: value HLK-PM01 -> LM338K; device HLK-PM01:HLK-PM01 -> REG1117:LM338K-MOLEX
- renumbered C11 to C4, C15 to C10, IC5 to IC1, IC6 to IC2
Connections:
- removed net HIGH_TEMPERATURE_1: R28.1, R31.1
- net !SHORT_CIRCUIT_DETECTED!: now also OK2.E, OK4.E, Q4.C, R14.2, R31.2; no longer OK1.E, OK3.E, Q2.C, R35.2, R46.2
- net !VOUT1_POWER_OFF!: now also IC3B.OUT, R34.2, R35.1, R43.2, R44.1, R45.1; no longer IC4B.OUT, R16.1, R23.2, R25.2, R33.1, R34.1
- net !VOUT1_POWER_ON!: now also IC3B.-IN, R33.2, R37.1, R38.2; no longer IC4B.-IN, R18.1, R19.2, R24.2
- net !VOUT1_POWER_ON!1: now also OK2.COL, R13.1; no longer OK1.COL, R11.1
- net !VOUT1_POWER_ON!2: now also OK1.COL, R11.1; no longer OK2.COL, R36.1
- net !VOUT1_POWER_ON!3: now also OK4.COL, R30.1; no longer OK3.COL, R44.1
- net !VOUT1_POWER_ON!4: now also OK3.COL, R28.1; no longer OK4.COL, R48.1
- net +12V: now also D4.C, IC3P.V+, Q5.E, R13.2, R19.E, R30.2, R37.2, R39.2, R40.2, RT3.2, U2.VO+; no longer D1.C, IC4P.V+, Q4.E, R18.2, R20.2, R36.2, R44.2, R48.2, R8.E, RT2.2, U3.VO+
- net 0V_A: now also R3.2; no longer R2.2
- net 0V_B: now also U2.AC2; no longer U3.AC2
- net 127V_A: now also R3.1; no longer R2.1
- net 127V_B: now also U2.AC1; no longer U3.AC1
- net 12V_AUX1: now also D1.C, R2.E, R6.1; no longer D9.C, R45.1, R7.E
- net 12V_AUX2: now also D5.C, R16.E, R17.E, R22.1; no longer D10.C, R40.E, R5.E, R50.1
- net C_FULL_1: now also C1.+, C2.1, K12.S, R4.2, R6.2; no longer C7.+, C8.1, K22.S, R3.2, R45.2
- net C_FULL_2: now also C7.+, C8.1, D6.C, K22.S, R18.2, R22.2, RT2.1, U3.VIN; no longer C12.+, C13.1, D4.C, K12.S, R41.2, R50.2, RT4.1, U2.VIN
- net GND1: now also C1.-, C2.2, C3.-, D1.A, R10.A, R10.S, R2.A, R5.1; no longer C7.-, C8.2, C9.-, D9.A, R14.A, R14.S, R33.2, R4.1, R7.A
- net GND2: now also C7.-, C8.2, C9.-, D5.A, R16.A, R17.A, R20.1; no longer C12.-, C13.2, C14.-, D10.A, R40.A, R42.1, R5.A
- net HIGH_TEMPERATURE: now also IC3A.OUT, R25.2, R39.1, R42.1; no longer IC4A.OUT, R12.2
- net N$1: now also K12.P; no longer K22.P
- net N$12: now also D10.C, R36.1; no longer D7.C, R29.1
- net N$13: now also R36.2; no longer R29.2
- net N$14: now also R33.1; no longer R24.1
- net N$15: now also R9.E; no longer R13.E
- net N$16: now also C3.+, R10.E, R9.A, R9.S; no longer C9.+, R13.A, R13.S, R14.E
- net N$18: now also R4.1, R5.2; no longer R3.1, R4.2
- net N$19: now also R8.1; no longer R10.1
- net N$2: now also D4.A, K11.2; no longer D1.A, K21.2
- net N$20: now also OK2.A, R8.2; no longer OK1.A, R10.2
- net N$21: now also IC3B.+IN, Q4.E, R40.1, R41.2, R43.1; no longer IC4B.+IN, Q2.E, R20.1, R21.2, R23.1
- net N$22: now also Q4.B, R35.2; no longer Q2.B, R16.2
- net N$25: now also R2.S; no longer R7.S
- net N$26: now also D6.A, D7.C, U3.VOUT; no longer D4.A, D5.C, U2.VOUT
- net N$27: now also C9.+, D7.A, U3.GND; no longer C14.+, D5.A, U2.GND
- net N$29: now also K22.P, RT2.2; no longer K12.P, RT4.2
- net N$3: now also R34.1; no longer R25.1
- net N$32: now also Q5.B, R42.2; no longer Q4.B, R31.2
- net N$33: now also K21.2, Q2.C; no longer K11.2, Q7.C
- net N$35: now also IC3A.-IN, R21.E, R21.S, RT3.1; no longer IC4A.-IN, R9.E, R9.S, RT2.1
- net N$36: now also IC3A.+IN, R19.S, R25.1; no longer IC4A.+IN, R12.1, R8.S
- net N$37: now also R7.1; no longer R37.1
- net N$38: now also D9.C, Q5.C; no longer D6.C, Q4.C
- net N$39: now also OK1.A, R7.2; no longer OK2.A, R37.2
- net N$4: now also R15.2; no longer R6.2
- net N$40: now also Q2.B, R32.2; no longer Q7.B, R39.2
- net N$41: now also R18.1, R20.2; no longer R41.1, R42.2
- net N$42: now also R24.1; no longer R43.1
- net N$43: now also R16.S; no longer R40.S
- net N$44: now also OK4.A, R24.2; no longer OK3.A, R43.2
- net N$45: now also R23.1; no longer R47.1
- net N$46: now also OK3.A, R23.2; no longer OK4.A, R47.2
- net N$47: now also OK3.E, R29.2, R32.1; no longer OK4.E, R39.1, R49.2
- net N$48: now also OK1.E, R12.2, R15.1; no longer OK2.E, R38.2, R6.1
- net N$5: now also R17.S; no longer R5.S
- net N$7: now also R45.2; no longer R34.2
- net PE: now also D10.A, D9.A, IC3P.V-, Q2.E, R12.1, R14.1, R19.A, R21.A, R29.1, R31.1, R41.1, R44.2, U2.VO-; no longer D6.A, D7.A, IC4P.V-, Q7.E, R19.1, R21.1, R35.1, R46.1, R49.1, R8.A, R9.A, U3.VO-
Other:
- moved on the sheet: C7, C8, C9, D3, D4, D6, D7, D8, K1, K2, K3, K4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

Commit message: Schematic 2.1 (better organization)
Parts:
- added C11, C12, C15: 100nF x 50V, rcl:C-EUC0805
- added C13, C14: 10uF x 50V, rcl:CPOL-EU153CLV-0605
Connections:
- removed net +24V: VOLT1.P$1, VOLT2.P$1
- new net 0V: C11.2, C12.2
- net +12V: now also C15.1
- net 12V_AUX1: now also C11.1, C13.+, VOLT1.P$1
- net 12V_AUX2: now also C12.1, C14.+, VOLT2.P$1
- net GND1: now also C13.-
- net GND2: now also C14.-
- net PE: now also C15.2
Other:
- note added: "2.1"
- note added: "HEAT SINK TEMPERATURE MONITOR"
- note added: "ISOLATED RELAY DRIVER"
- note added: "ISOLATED TRIGGER PULSE"
- note added: "OUTPUT STATUS"
- note removed: "1"
- note removed: "2"
- note removed: "2.0"
- note removed: "3"
- note removed: "4"
- note removed: "5"
- note removed: "6"
- note removed: "OUTPUT STATUS USER INTERFACE"
- note removed: "TEMPERATURE MONITOR HEAT SINK"
- moved on the sheet: C10, C2, C3, C4, C9, D1, D2, D3, D5, D6, D7, F1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

Commit message: Working on at 2.1 schematic
Parts:
- added D11: 1N4148, diode:DIODE-SOD80C
- added X3: 22-23-2021, con-molex-PTR:22-23-2021
- D10, D4, D8, D9: device diode:DIODE-SOD523 -> diode:DIODE-SOD80C
- K1, K2, K3, K4: device relay:ZNS5448 -> relay:CQ1-12V
- R26, R9: device rcl:R-TRIMM64W -> pot:TRIM_EU-CA6V
Connections:
- net !VOUT1_POWER_OFF! renamed !VOUT_POWER_OFF!
- net 0V_B: now also X3-2.S
- net 127V_B: now also X3-1.S
- net N$12: now also D11.C
- net PE: now also D11.A
Other:
- moved on the sheet: K1, K2, K3, K4

Commit message: Schematic and PCB layout 2.1 updated
Parts:
- removed IC1: LM393D, linear:LM393D
- removed OK1: 4N33, optocoupler:4N33
- added U10: LM338K-MOLEX, REG1117:LM338K-MOLEX
- added U5: HLK-PM01, HLK-PM01:HLK-PM01
- B1, B2: value KBPC608 -> (none)
- C1: value 15.000uF x 50V -> (none)
- C10, C14, C3: value 10uF x 50V -> (none); device rcl:CPOL-EU153CLV-0605 -> rcl:C-EUC0805
- C11, C2: value 100nF x 50V -> (none)
- C12, C15, C5, C8: value 100nF x 50V -> (none); device rcl:C-EUC0805 -> rcl:CPOL-EU153CLV-0605
- C13, C4, C6: value 10uF x 50V -> (none)
- C7: value 15.000uF x 50V -> (none); device rcl:CPOL-EUE10-35 -> rcl:C-EUC0805
- C9: value 10uF x 50V -> (none); device rcl:CPOL-EU153CLV-0605 -> rcl:CPOL-EUE10-35
- D1, D5: value 12V / 0.5W -> (none)
- D10, D11, D4, D8, D9: value 1N4148 -> (none)
- D2, D3, D6, D7: value 1N4007 -> CGRM4007-G
- K1, K2, K3, K4: value 12VDC COIL -> CQ1-12V
- LED1: value Bicolor LED Common-Anode -> LED-BICOLOR-MOLEX3P
- Q1, Q2: value BC848 -> BC848SMD
- Q3, Q5, Q6: value BC858 -> BC858BSMD
- Q4: value BC848 -> BC848BSMD
- R1, R16, R17, R2: value 500k -> (none); device rcl:R-TRIMM64W -> rcl:R-TRIMM3202
- R10, R27: value 5K -> (none); device trimpot-molex2p:R-TRIMM -> rcl:R-EU_R0805
- R11, R28, R34, R36: value 1k (5%) -> (none)
- R12, R29, R44: value 100k (5%) -> (none)
- R13, R30: value 1k (5%) -> (none); device rcl:R-EU_R0805 -> rcl:R-TRIMM3202
- R14, R31: value 100k (5%) -> (none); device rcl:R-EU_R0805 -> trimpot-molex2p:R-TRIMM
- R15, R23, R24, R32, R33, R35, R39, R42, R45, R7, R8: value 10k (5%) -> (none)
- R18, R37, R38, R4, R40, R41: value 100k (1%) -> (none)
- R19, R21: value 10k -> (none); device rcl:R-TRIMM64W -> rcl:R-TRIMM3202
- R20, R5: value 33k (1%) -> (none)
- R22, R6: value 220R -> (none)
- R25: value 33k (5%) -> (none)
- R26, R9: value 500R -> (none); device pot:TRIM_EU-CA6V -> rcl:R-EU_R0805
- R43: value 220k (5%) -> (none)
- RT1, RT2: value 5R -> NTC-11MM
- RT3: value 10k -> NTC-MOLEX2P
- TR1, TR2: value 24VRMS -> TRAFO
- U1: value LM338K -> LM393D; device REG1117:LM338K-MOLEX -> linear:LM393D
- U2: value HLK-PM01 -> LM338K-MOLEX; device HLK-PM01:HLK-PM01 -> REG1117:LM338K-MOLEX
- U3: value LM338K -> 4N33; device REG1117:LM338K-MOLEX -> optocoupler:4N33
- renumbered IC2 to U6, IC3 to U7, OK2 to U4, OK3 to U8, OK4 to U9
Connections:
- removed net 0V: C11.2, C12.2
- net !SHORT_CIRCUIT_DETECTED!: now also R12.2, R29.2; no longer R14.2, R31.2
- net !VOUT1_POWER_ON!1: now also R11.1; no longer R13.1
- net !VOUT1_POWER_ON!2: now also R9.1, U3.COL; no longer OK1.COL, R11.1
- net !VOUT1_POWER_ON!3: now also R28.1; no longer R30.1
- net !VOUT1_POWER_ON!4: now also R26.1; no longer R28.1
- net +12V: now also C14.1, C7.1, C8.+, R26.2, R9.2, U5.VO+; no longer C15.1, C5.1, C6.+, R13.2, R30.2, U2.VO+
- net 0V_B: now also U5.AC2, X1-2.S; no longer U2.AC2, X3-2.S
- net 127V_B: now also U5.AC1, X1-1.S; no longer U2.AC1, X3-1.S
- net 12V_AUX1: now also C3.1, C4.+, U1P.V+; no longer C11.1, C13.+, IC1P.V+
- net 12V_AUX2: now also C11.1, C12.+; no longer C12.1, C14.+
- net C_FULL_1: now also U2.VIN; no longer U1.VIN
- net C_FULL_2: now also C10.1, C9.+, U10.VIN; no longer C7.+, C8.1, U3.VIN
- net GND1: now also C3.2, C5.-, C6.-, R14.A, R14.S, U1P.V-, U3.C, X2-2.S; no longer C13.-, C3.-, IC1P.V-, OK1.C, R10.A, R10.S, X1-2.S
- net GND2: now also C10.2, C11.2, C12.-, C13.-, C15.-, R31.A, R31.S, X3-2.S; no longer C10.-, C14.-, C7.-, C8.2, R27.A, R27.S, X2-2.S
- net N$12: now also D9.C; no longer D10.C
- net N$15: now also C6.+, R13.E, U2.VOUT; no longer C4.+, R9.E, U1.VOUT
- net N$16: now also C5.+, R13.A, R13.S, R14.E, U2.GND; no longer C3.+, R10.E, R9.A, R9.S, U1.GND
- net N$17: now also X2-1.S; no longer X1-1.S
- net N$18: now also U1B.+IN; no longer IC1B.+IN
- net N$19: now also R7.1, U1A.OUT; no longer IC1A.OUT, R8.1
- net N$20: now also R7.2; no longer R8.2
- net N$25: now also U1A.-IN; no longer IC1A.-IN
- net N$26: now also C15.+, R30.E, U10.VOUT; no longer C10.+, R26.E, U3.VOUT
- net N$27: now also C13.+, R30.A, R30.S, R31.E, U10.GND; no longer C9.+, R26.A, R26.S, R27.E, U3.GND
- net N$28: now also X3-1.S; no longer X2-1.S
- net N$37: now also R8.1, U1B.OUT; no longer IC1B.OUT, R7.1
- net N$38: now also D10.C; no longer D9.C
- net N$39: now also R8.2, U3.A; no longer OK1.A, R7.2
- net N$42: now also R23.1; no longer R24.1
- net N$44: now also R23.2; no longer R24.2
- net N$45: now also R24.1; no longer R23.1
- net N$46: now also R24.2; no longer R23.2
- net N$47: now also R27.2; no longer R29.2
- net N$48: now also R10.2, U3.E; no longer OK1.E, R12.2
- net N$6: now also U1B.-IN; no longer IC1B.-IN
- net PE: now also C14.2, C7.2, C8.-, R10.1, R27.1, U5.VO-; no longer C15.2, C5.2, C6.-, R14.1, R31.1, U2.VO-
- net VOUT_1: now also U1A.+IN; no longer IC1A.+IN, U6A.+IN
- net VOUT_2: now also U6A.+IN
Other:
- note added: "127V OR 220V AC INPUT VOLTAGE SELECT"
- note added: "2.2"
- note removed: "127V OR 220V AC INPUTY SELECT"
- note removed: "2.1"
- moved on the sheet: C11, C13, C4, C6, C9, D10, D11, D9, R11, R12, R23, R24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
